File: hardware/sounddecoder-esp32-s3-wroom-1/sounddecoder-esp32-s3-wroom-1.kicad_sch (KiCad schematic)
At the start: 7 parts, among them J1 Input power, U1 ESP32-WROOM-32D, U2 IS25WP256D-xM, U3 MAX98357A, U4 DRV8871DDA, U5 LM2594M-5.0, U6 AMS1117-3.3

Commit message: Many updates
Parts:
- removed U1: ESP32-WROOM-32D, RF_Module:ESP32-WROOM-32D, symbol RF_Module:ESP32-WROOM-32D
- added U7: ESP32-S3-WROOM-1, RF_Module:ESP32-S3-WROOM-1, symbol RF_Module:ESP32-S3-WROOM-1
Connections:
- net +3.3V: now also U7.2 (3V3)
- net GND: now also U7.1 (GND), U7.40 (GND), U7.41 (GND)
Changed lines of the file:
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@@
 	(symbol
 		(lib_id "power:GND")
-		(at 54.61 166.37 0)
+		(at 46.99 149.86 0)
 		(unit 1)
 		(exclude_from_sim no)
@@
 		(fields_autoplaced yes)
 		(property "Reference" "#PWR012"
-			(at 54.61 172.72 0)
+			(at 46.99 156.21 0)
 			(effects
 				(font
@@
 		)
 		(property "Value" "GND"
-			(at 54.61 171.45 0)
+			(at 46.99 154.94 0)
 			(effects
 				(font
@@
 		)
 		(property "Footprint" ""
-			(at 54.61 166.37 0)
+			(at 46.99 149.86 0)
 			(effects
 				(font
@@
 		)
 		(property "Datasheet" ""
-			(at 54.61 166.37 0)
+			(at 46.99 149.86 0)
 			(effects
 				(font
@@
 		)
 		(property "Description" "Power symbol creates a global label with name \"GND\" , ground"
-			(at 54.61 166.37 0)
+			(at 46.99 149.86 0)
 			(effects
 				(font
@@
 	(symbol
 		(lib_id "power:+3.3V")
-		(at 54.61 95.25 0)
+		(at 46.99 93.98 0)
 		(unit 1)
 		(exclude_from_sim no)
@@
 		(fields_autoplaced yes)
 		(property "Reference" "#PWR05"
-			(at 54.61 99.06 0)
+			(at 46.99 97.79 0)
 			(effects
 				(font
@@
 		)
 		(property "Value" "+3.3V"
-			(at 54.61 90.17 0)
+			(at 46.99 88.9 0)
 			(effects
 				(font
@@
 		)
 		(property "Footprint" ""
-			(at 54.61 95.25 0)
+			(at 46.99 93.98 0)
 			(effects
 				(font
@@
 		)
 		(property "Datasheet" ""
-			(at 54.61 95.25 0)
+			(at 46.99 93.98 0)
 			(effects
 				(font
@@
 		)
 		(property "Description" "Power symbol creates a global label with name \"+3.3V\""
-			(at 54.61 95.25 0)
+			(at 46.99 93.98 0)
 			(effects
 				(font
@@
 	)
 	(symbol
-		(lib_id "RF_Module:ESP32-WROOM-32D")
-		(at 54.61 130.81 0)
-		(unit 1)
-		(exclude_from_sim no)
-		(in_bom yes)
-		(on_board yes)
-		(dnp no)
-		(fields_autoplaced yes)
-		(property "Reference" "U1"
-			(at 56.7533 92.71 0)
-			(effects
-				(font
-					(size 1.27 1.27)
-				)
-				(justify left)
-			)
-		)
-		(property "Value" "ESP32-WROOM-32D"
-			(at 56.7533 95.25 0)
-			(effects
-				(font
-					(size 1.27 1.27)
-				)
-				(justify left)
-			)
-		)
-		(property "Footprint" "RF_Module:ESP32-WROOM-32D"
-			(at 71.12 165.1 0)
-			(effects
-				(font
-					(size 1.27 1.27)
-				)
-				(hide yes)
-			)
-		)
-		(property "Datasheet" "https://www.espressif.com/sites/default/files/documentation/esp32-wroom-32d_esp32-wroom-32u_datasheet_en.pdf"
-			(at 46.99 129.54 0)
-			(effects
-				(font
-					(size 1.27 1.27)
-				)
-				(hide yes)
-			)
-		)
-		(property "Description" "RF Module, ESP32-D0WD SoC, Wi-Fi 802.11b/g/n, Bluetooth, BLE, 32-bit, 2.7-3.6V, onboard antenna, SMD"
-			(at 54.61 130.81 0)
-			(effects
-				(font
-					(size 1.27 1.27)
-				)
-				(hide yes)
-			)
-		)
-		(pin "12"
-		)
-		(pin "21"
-		)
-		(pin "15"
-		)
-		(pin "22"
-		)
-		(pin "38"
-		)
-		(pin "10"
-		)
-		(pin "37"
-		)
-		(pin "5"
-		)
-		(pin "39"
-		)
-		(pin "6"
-		)
-		(pin "8"
-		)
-		(pin "9"
-		)
-		(pin "2"
-		)
-		(pin "18"
-		)
-		(pin "4"
-		)
-		(pin "7"
-		)
-		(pin "20"
-		)
-		(pin "33"
-		)
-		(pin "35"
-		)
-		(pin "17"
-		)
-		(pin "13"
-		)
-		(pin "29"
-		)
-		(pin "26"
-		)
-		(pin "11"
-		)
-		(pin "23"
-		)
-		(pin "32"
-		)
-		(pin "27"
-		)
-		(pin "34"
-		)
-		(pin "14"
-		)
-		(pin "16"
-		)
-		(pin "25"
-		)
-		(pin "19"
-		)
-		(pin "3"
-		)
-		(pin "31"
-		)
-		(pin "30"
-		)
-		(pin "1"
-		)
-		(pin "36"
-		)
-		(pin "24"
-		)
-		(pin "28"
-		)
-		(instances
-			(project ""
-				(path "/d1fe0542-ce5f-402b-bc04-d653d7366528"
-					(reference "U1")
-					(unit 1)
-				)
-			)
-		)
-	)
-	(symbol
 		(lib_id "power:+3.3V")
 		(at 140.97 116.84 0)
@@
 					(unit 1)
 				)
+			)
+		)
+	)
+	(symbol
+		(lib_id "RF_Module:ESP32-S3-WROOM-1")
+		(at 46.99 121.92 0)
+		(unit 1)
+		(exclude_from_sim no)
+		(in_bom yes)
+		(on_board yes)
+		(dnp no)
+		(fields_autoplaced yes)
+		(property "Reference" "U7"
+			(at 49.1333 91.44 0)
+			(effects
+				(font
+					(size 1.27 1.27)
+				)
+				(justify left)
+			)
+		)
+		(property "Value" "ESP32-S3-WROOM-1"
+			(at 49.1333 93.98 0)
+			(effects
+				(font
+					(size 1.27 1.27)
+				)
+				(justify left)
+			)
+		)
+		(property "Footprint" "RF_Module:ESP32-S3-WROOM-1"
+			(at 46.99 119.38 0)
+			(effects
+				(font
+					(size 1.27 1.27)
+				)
+				(hide yes)
+			)
+		)
+		(property "Datasheet" "https://www.espressif.com/sites/default/files/documentation/esp32-s3-wroom-1_wroom-1u_datasheet_en.pdf"
+			(at 46.99 121.92 0)
+			(effects
+				(font
+					(size 1.27 1.27)
+				)
+				(hide yes)
+			)
+		)
+		(property "Description" "RF Module, ESP32-S3 SoC, Wi-Fi 802.11b/g/n, Bluetooth, BLE, 32-bit, 3.3V, onboard antenna, SMD"
+			(at 46.99 121.92 0)
+			(effects
+				(font
+					(size 1.27 1.27)
+				)
+				(hide yes)
+			)
+		)
+		(pin "19"
+		)
+		(pin "36"
+		)
+		(pin "14"
+		)
+		(pin "13"
+		)
+		(pin "11"
+		)
+		(pin "9"
+		)
+		(pin "8"
+		)
+		(pin "25"
+		)
+		(pin "33"
+		)
+		(pin "22"
+		)
+		(pin "10"
+		)
+		(pin "20"
+		)
+		(pin "32"
+		)
+		(pin "6"
+		)
+		(pin "12"
+		)
+		(pin "35"
+		)
+		(pin "3"
+		)
+		(pin "16"
+		)
+		(pin "34"
+		)
+		(pin "24"
+		)
+		(pin "26"
+		)
+		(pin "30"
+		)
+		(pin "31"
+		)
+		(pin "41"
+		)
+		(pin "7"
+		)
+		(pin "15"
+		)
+		(pin "4"
+		)
+		(pin "5"
+		)
+		(pin "27"
+		)
+		(pin "40"
+		)
+		(pin "39"
+		)
+		(pin "38"
+		)
+		(pin "18"
+		)
+		(pin "2"
+		)
+		(pin "29"
+		)
+		(pin "28"
+		)
+		(pin "37"
+		)
+		(pin "17"
+		)
+		(pin "23"
+		)
+		(pin "21"
+		)
+		(pin "1"
+		)
+		(instances
+			(project ""
+				(path "/d1fe0542-ce5f-402b-bc04-d653d7366528"
+					(reference "U7")
+					(unit 1)
+				)

Commit message: Many updates
Parts:
- removed U5: LM2594M-5.0, Package_SO:SOIC-8_3.9x4.9mm_P1.27mm, symbol Regulator_Switching:LM2594M-5.0
- added C1, C10, C9: 0.1uF, Capacitor_SMD:C_0805_2012Metric, symbol Device:C
- added C11: 22uF, Capacitor_SMD:C_0805_2012Metric, symbol Device:C
- added C2: 47uF, Capacitor_SMD:C_0805_2012Metric, symbol Device:C
- added C3: 105, symbol Device:C
- added C4: 470uF, symbol Device:C_Polarized
- added C5: 220uF, Capacitor_Tantalum_SMD:CP_EIA-7343-20_Kemet-V_HandSolder, symbol Device:C_Polarized
- added C6: 22uF, Capacitor_Tantalum_SMD:CP_EIA-3216-10_Kemet-I_HandSolder, symbol Device:C_Polarized
- added C7: 10uF, symbol Device:C
- added C8: 0.1uF, symbol Device:C
- added D1: 1N5825, Diode_THT:D_DO-201AD_P15.24mm_Horizontal, symbol Diode:1N5822
- added J2: Physical outputs, symbol Connector_Generic:Conn_02x07_Row_Letter_Last
- added J3: Motor, symbol Connector_Generic:Conn_01x02
- added J4: Speaker, symbol Connector_Generic:Conn_01x02
- added J5: UART, Connector_PinSocket_2.54mm:PinSocket_1x04_P2.54mm_Horizontal, symbol Connector:Conn_01x04_Pin
- added L1: 47uh/L39, Inductor_SMD:L_Bourns_SRP1245A, symbol Device:L
- added R1: 15k, symbol Device:R
- added R2: 10k, symbol Device:R
- added U1: LM2596S-5, Package_TO_SOT_SMD:TO-263-5_TabPin3, symbol Regulator_Switching:LM2596S-5
- added U8: ULN2003A, symbol Transistor_Array:ULN2003A
Connections:
- net +3.3V: now also U3.4 (~{SD_MODE}), C10.1, C11.1, C6.1, C7.1, C8.1, C9.1, J5.1 (Pin_1), R2.1; no longer U4.5 (VM)
- net GND: now also J1.2 (Pin_2), U3.17 (PAD), U3.2 (GAIN_SLOT), C1.2, C10.2, C11.2, C2.2, C3.2, C4.2, C5.2, C6.2, C7.2, C8.2, C9.2, D1.2 (A), J5.4 (Pin_4), R1.2, U1.3 (GND), U1.5 (~{ON}/OFF), U8.8 (GND); no longer J1.1 (Pin_1)
- net at U3.1 (DIN): now also U7.19 (IO11)
- net at U3.10 (OUTN): now also J4.2 (Pin_2)
- net at U3.14 (LRCLK): now also U7.21 (IO13)
- net at U3.16 (BCLK): now also U7.20 (IO12)
- net at U3.9 (OUTP): now also J4.1 (Pin_1)
- net +5V: now reaches U6.3 (VI)
- net +5V: now also C5.1, J2.1b (Pin_1b), J2.2b (Pin_2b), J2.3b (Pin_3b), J2.4b (Pin_4b), J2.5b (Pin_5b), J2.6b (Pin_6b), J2.7b (Pin_7b), L1.2, U1.4 (FB), U8.9 (COM)
- net at U7.12 (IO8): now also U2.7 (~{CE})
- net at U7.17 (IO9): now also U2.9 (~{WP}/IO2)
- net at U7.18 (IO10): now also U2.1 (~{HOLD}/IO3)
- net at U7.24 (IO47): now also U8.6 (I6)
- net at U7.25 (IO48): now also U8.7 (I7)
- net at U7.3 (EN): now also R2.2
- net at U7.31 (IO38): now also U8.1 (I1)
- net at U7.32 (IO39): now also U8.2 (I2)
- net at U7.33 (IO40): now also U8.3 (I3)
- net at U7.34 (IO41): now also U8.4 (I4)
- net at U7.35 (IO42): now also U8.5 (I5)
- net at U7.36 (RXD0): now also J5.3 (Pin_3)
- net at U7.37 (TXD0): now also J5.2 (Pin_2)
- net at U7.38 (IO2): now also U4.3 (IN1)
- net MOTOR_SENSE: now reaches U7.39 (IO1)
- net MOTOR_SENSE: now also U4.4 (ILIM), R1.1
- net at U7.4 (IO4): now also U4.2 (IN2)
- net at U7.5 (IO5): now also U2.15 (SI/IO0)
- net at U7.6 (IO6): now also U2.8 (SO/IO1)
- net at U7.7 (IO7): now also U2.16 (SCK)
- net at U4.6 (OUT1): now also J3.1 (Pin_1)
- net at U4.8 (OUT2): now also J3.2 (Pin_2)
- new net: J2.7a (Pin_7a), U8.10 (O7)
- new net: J2.6a (Pin_6a), U8.11 (O6)
- new net: J2.5a (Pin_5a), U8.12 (O5)
- new net: J2.4a (Pin_4a), U8.13 (O4)
- new net: D1.1 (K), L1.1, U1.2 (OUT)
- new net BackLED: J2.3a (Pin_3a), U8.14 (O3)
- new net FwdLED: J2.2a (Pin_2a), U8.15 (O2)
- new net Smoke: J2.1a (Pin_1a), U8.16 (O1)
- new net VCC: C1.1, C2.1, C3.1, C4.1, J1.1 (Pin_1), U1.1 (VIN), U4.5 (VM)
- no-connect marks 0 -> 7
Other:
- moved on the sheet: J1, U2, U3, U4, U7

Commit message: Created PCB
Parts:
- removed J2: Physical outputs, symbol Connector_Generic:Conn_02x07_Row_Letter_Last
- removed U2: IS25WP256D-xM, Package_SO:SOIC-16W_7.5x10.3mm_P1.27mm, symbol Memory_Flash:IS25WP256D-xM
- added J10: AUX1, TerminalBlock:TerminalBlock_Xinya_XY308-2.54-2P_1x02_P2.54mm_Horizontal, symbol Connector_Generic:Conn_01x02
- added J11: AUX2, TerminalBlock:TerminalBlock_Xinya_XY308-2.54-2P_1x02_P2.54mm_Horizontal, symbol Connector_Generic:Conn_01x02
- added J12: AUX3, TerminalBlock:TerminalBlock_Xinya_XY308-2.54-2P_1x02_P2.54mm_Horizontal, symbol Connector_Generic:Conn_01x02
- added J13: AUX4, TerminalBlock:TerminalBlock_Xinya_XY308-2.54-2P_1x02_P2.54mm_Horizontal, symbol Connector_Generic:Conn_01x02
- added J6: Conn_01x03_Pin, Connector_PinHeader_1.00mm:PinHeader_1x03_P1.00mm_Vertical, symbol Connector:Conn_01x03_Pin
- added J7: Smoke, TerminalBlock:TerminalBlock_Xinya_XY308-2.54-2P_1x02_P2.54mm_Horizontal, symbol Connector_Generic:Conn_01x02
- added J8: FwdLED, TerminalBlock:TerminalBlock_Xinya_XY308-2.54-2P_1x02_P2.54mm_Horizontal, symbol Connector_Generic:Conn_01x02
- added J9: BackLED, TerminalBlock:TerminalBlock_Xinya_XY308-2.54-2P_1x02_P2.54mm_Horizontal, symbol Connector_Generic:Conn_01x02
- added U5: W25Q256, Package_SON:WSON-8-1EP_6x5mm_P1.27mm_EP3.4x4.3mm, symbol Memory_Flash:W25Q128JVP
- C1, C10, C11, C9: footprint Capacitor_SMD:C_0805_2012Metric -> Capacitor_SMD:C_0805_2012Metric_Pad1.18x1.45mm_HandSolder
- C2: footprint Capacitor_SMD:C_0805_2012Metric -> Capacitor_SMD:CP_Elec_6.3x5.4; symbol Device:C -> Device:C_Polarized
- C3: value 105 -> 0.1uF; footprint (none) -> Capacitor_SMD:C_0805_2012Metric_Pad1.18x1.45mm_HandSolder
- C4: footprint (none) -> Capacitor_SMD:CP_Elec_10x10.5
- C5: footprint Capacitor_Tantalum_SMD:CP_EIA-7343-20_Kemet-V_HandSolder -> Capacitor_SMD:C_Elec_6.3x7.7
- C6: footprint Capacitor_Tantalum_SMD:CP_EIA-3216-10_Kemet-I_HandSolder -> Capacitor_SMD:CP_Elec_4x5.4
- C7, C8: footprint (none) -> Capacitor_SMD:C_0805_2012Metric_Pad1.18x1.45mm_HandSolder
- D1: value 1N5825 -> SS54; footprint Diode_THT:D_DO-201AD_P15.24mm_Horizontal -> Diode_SMD:D_SMA_Handsoldering
- J1, J3, J4: footprint (none) -> TerminalBlock:TerminalBlock_Xinya_XY308-2.54-2P_1x02_P2.54mm_Horizontal
- R1, R2: footprint (none) -> Resistor_SMD:R_0805_2012Metric_Pad1.20x1.40mm_HandSolder
- U8: footprint (none) -> Package_SO:SO-16_3.9x9.9mm_P1.27mm
Connections:
- net +3.3V: now also J6.3 (Pin_3), U5.8 (VCC)
- net +5V: now also J10.1 (Pin_1), J11.1 (Pin_1), J12.1 (Pin_1), J13.1 (Pin_1), J7.1 (Pin_1), J8.1 (Pin_1), J9.1 (Pin_1)
- net BackLED: now also J9.2 (Pin_2)
- net FwdLED: now also J8.2 (Pin_2)
- net GND: now also J6.1 (Pin_1), U5.4 (GND), U5.9 (EP); no longer U3.2 (GAIN_SLOT)
- net Smoke: now also J7.2 (Pin_2)
- net Sound2: now reaches J4.2 (Pin_2), U3.10 (OUTN)
- net Sound1: now reaches J4.1 (Pin_1), U3.9 (OUTP)
- net at U8.1 (I1): now also U7.24 (IO47); no longer U7.31 (IO38)
- net at U8.10 (O7): now also J13.2 (Pin_2)
- net at U8.11 (O6): now also J12.2 (Pin_2)
- net at U8.12 (O5): now also J11.2 (Pin_2)
- net at U8.13 (O4): now also J10.2 (Pin_2)
- net at U8.2 (I2): now also U7.25 (IO48); no longer U7.32 (IO39)
- net at U8.3 (I3): now also U7.35 (IO42); no longer U7.33 (IO40)
- net at U8.5 (I5): now also U7.33 (IO40); no longer U7.35 (IO42)
- net at U8.6 (I6): now also U7.32 (IO39); no longer U7.24 (IO47)
- net at U8.7 (I7): now also U7.31 (IO38); no longer U7.25 (IO48)
- net UART-TX: now reaches J5.2 (Pin_2), U7.37 (TXD0)
- net UART-RX: now reaches J5.3 (Pin_3), U7.36 (RXD0)
- net Out5V: now reaches D1.1 (K), L1.1, U1.2 (OUT)
- net MEM_IO3: now reaches U7.10 (IO17)
- net MEM_IO3: now also U5.7 (~{HOLD}/~{RESET}/IO_{3})
- net MEM_SCK: now reaches U7.11 (IO18)
- net MEM_SCK: now also U5.6 (CLK)
- net MEM_IO0: now reaches U7.12 (IO8)
- net MEM_IO0: now also U5.5 (DI/IO_{0})
- net MEM_CE: now reaches U7.7 (IO7)
- net MEM_CE: now also U5.1 (~{CS})
- net MEM_IO1: now reaches U7.8 (IO15)
- net MEM_IO1: now also U5.2 (DO/IO_{1})
- net MEM_IO2: now reaches U7.9 (IO16)
- net MEM_IO2: now also U5.3 (~{WP}/IO_{2})
- net MOTOR1: now reaches J3.1 (Pin_1), U4.6 (OUT1)
- net MOTOR2: now reaches J3.2 (Pin_2), U4.8 (OUT2)
- new net SND_GAIN: J6.2 (Pin_2), U3.2 (GAIN_SLOT)
Other:
- moved on the sheet: C7, C8, C9, J3, J4, U8

Commit message: Started working on board v2
Parts:
- added C12: 1uF, Capacitor_SMD:C_0805_2012Metric_Pad1.18x1.45mm_HandSolder, symbol Device:C
- added J2: Boot, Connector_PinHeader_1.00mm:PinHeader_1x03_P1.00mm_Vertical, symbol Connector:Conn_01x03_Pin
- D1: footprint Diode_SMD:D_SMA_Handsoldering -> Diode_SMD:D_SMC
- U5: footprint Package_SON:WSON-8-1EP_6x5mm_P1.27mm_EP3.4x4.3mm -> Package_SON:WSON-8-1EP_8x6mm_P1.27mm_EP3.4x4.3mm
Connections:
- net +3.3V: now also J2.1 (Pin_1)
- net GND: now also C12.1, J2.3 (Pin_3)
- net at R2.2, U7.3 (EN): now also C12.2
- net at U7.27 (IO0): now also J2.2 (Pin_2)
- net MOTOR_SENSE: no longer names the net of R1.1, U4.4 (ILIM)
- net MOTOR_SENSE: no longer U7.39 (IO1)
- no-connect marks 7 -> 6
Other:
- moved on the sheet: C10, C11, R2
