File: hardware/sounddecoder-esp32-s3-wroom-2/sounddecoder-esp32-s3-wroom-2.kicad_pcb (KiCad board)
At the start: 4 copper layers, 42.5 x 59.8 mm, 34 parts, among them J1 Input power, J10 AUX1, J11 AUX2, J12 AUX3, J13 AUX4, J3 Motor, J4 Speaker, J5 DEBUG, J6 Conn_01x03_Pin, J7 Smoke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

Commit message: Finished v2 board
Parts:
- moved U8 1.08 mm to (97.3, 101.0)
- turned C5 to 90 degrees
Connections:
- U7 pad 19: unconnected-(U7-IO11-Pad19) -> /OUT7
- U7 pad 20: unconnected-(U7-IO12-Pad20) -> /OUT6
- U7 pad 21: unconnected-(U7-IO13-Pad21) -> /OUT5
- U7 pad 22: unconnected-(U7-IO14-Pad22) -> /OUT4
- U7 pad 23: unconnected-(U7-IO21-Pad23) -> /OUT3
- U7 pad 24: /OUT1 -> /OUT2
- U7 pad 25: /OUT2 -> /OUT1
- U7 pad 31: /OUT7 -> unconnected-(U7-IO38-Pad31)
- U7 pad 32: /OUT6 -> unconnected-(U7-MTCK/IO39-Pad32)
- U7 pad 33: /OUT5 -> unconnected-(U7-MTDO/IO40-Pad33)
- U7 pad 34: /OUT4 -> unconnected-(U7-MTDI/IO41-Pad34)
- U7 pad 35: /OUT3 -> unconnected-(U7-MTMS/IO42-Pad35)
Routing:
- net /MOTOR_SENSE: track 22.6 -> 73.8 mm
- net /MOTOR_IN1: track 16.4 -> 66.7 mm
- net +3.3V: track 5.57 -> 41.5 mm
- net +5V: track 28.1 -> 61.1 mm, vias 1 -> 5
- net /MOTOR_IN2: track 23.2 -> 55.5 mm
- net /Smoke: track 0.00 -> 30.4 mm, vias 0 -> 1
- net Net-(J13-Pin_2): track 1.02 -> 27.0 mm, vias 0 -> 1
- net /FwdLED: track 0.00 -> 24.7 mm, vias 0 -> 1
- net Net-(J12-Pin_2): track 0.00 -> 20.8 mm, vias 0 -> 1
- net /BackLED: track 0.00 -> 19.4 mm, vias 0 -> 1
- net /UART-TX: track 8.24 -> 27.2 mm
- net /UART-RX: track 8.19 -> 25.6 mm
- net Net-(J10-Pin_2): track 0.00 -> 15.9 mm, vias 0 -> 1
- net Net-(J11-Pin_2): track 0.00 -> 15.6 mm, vias 0 -> 1
- net /AUDIO_LRCLK: track 0.00 -> 14.3 mm, vias 0 -> 2
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- added copper zone on F.Cu, net +5V
