File: hardware/sounddecoder-esp32-s3-wroom-2/sounddecoder-esp32-s3-wroom-2.kicad_sch (KiCad schematic)
At the start: 34 parts, among them J1 Input power, J10 AUX1, J11 AUX2, J12 AUX3, J13 AUX4, J3 Motor, J4 Speaker, J5 DEBUG, J6 Conn_01x03_Pin, J7 Smoke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

Commit message: Finished v2 board
Connections:
- net OUT1: now also U7.25 (IO48); no longer U7.24 (IO47)
- net OUT2: now also U7.24 (IO47); no longer U7.25 (IO48)
- net OUT3: now also U7.23 (IO21); no longer U7.35 (MTMS/IO42)
- net OUT4: now also U7.22 (IO14); no longer U7.34 (MTDI/IO41)
- net OUT5: now also U7.21 (IO13); no longer U7.33 (MTDO/IO40)
- net OUT6: now also U7.20 (IO12); no longer U7.32 (MTCK/IO39)
- net OUT7: now also U7.19 (IO11); no longer U7.31 (IO38)
