File: hardware/sounddecoder-esp32-s3-wroom-2-micro/sounddecoder-esp32-s3-wroom-2-micro.kicad_pcb (KiCad board)
At the start: 4 copper layers, 22.5 x 48.3 mm, 48 parts, among them J1 Pins, J2 Conn_01x02_Pin, J3 TrackRight, J4 Smoke_Pin, J5 TrackLeft, U1 TPS54302, U2 DRV8235, U3 MAX98357A, U7 ESP32-S3-WROOM-2, U8 ULN2003A

Commit message: Added support of DRV8235 motor driver
Connections:
- U2 pad 12: /MOTOR_IN1 -> unconnected-(U2-PH/IN2-Pad12)
- U2 pad 13: /MOTOR_IN2 -> unconnected-(U2-EN/IN1-Pad13)
- U7 pad 38: /MOTOR_IN1 -> unconnected-(U7-IO2-Pad38)
- U7 pad 4: /MOTOR_IN2 -> unconnected-(U7-IO4-Pad4)
Routing:
- net /MOTOR_IN1: track 43.8 -> 0.00 mm, vias 4 -> 0
- net /MOTOR_IN2: track 41.7 -> 0.00 mm, vias 4 -> 0
Changed lines of the file:
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@@
 	(net 28 "/AUDIO_BCLK")
 	(net 29 "/AUDIO_LRCLK")
-	(net 30 "/MOTOR_IN1")
-	(net 31 "/MOTOR_IN2")
+	(net 30 "unconnected-(U2-EN{slash}IN1-Pad13)")
+	(net 31 "unconnected-(U2-PH{slash}IN2-Pad12)")
 	(net 32 "/SOUND2")
 	(net 33 "unconnected-(U7-IO15-Pad8)")
@@
 	(net 71 "/Track_Left")
 	(net 72 "Net-(C3-Pad1)")
+	(net 73 "unconnected-(U7-IO2-Pad38)")
+	(net 74 "unconnected-(U7-IO4-Pad4)")
 	(footprint "Inductor_SMD:L_Chilisin_BMRA00050530"
 		(layer "F.Cu")
@@
 			(size 1.5 0.9)
 			(layers "F.Cu" "F.Mask" "F.Paste")
-			(net 31 "/MOTOR_IN2")
+			(net 74 "unconnected-(U7-IO4-Pad4)")
 			(pinfunction "IO4")
-			(pintype "bidirectional")
+			(pintype "bidirectional+no_connect")
 		)
 		(pad "5" smd rect
@@
 			(size 1.5 0.9)
 			(layers "F.Cu" "F.Mask" "F.Paste")
-			(net 30 "/MOTOR_IN1")
+			(net 73 "unconnected-(U7-IO2-Pad38)")
 			(pinfunction "IO2")
-			(pintype "bidirectional")
+			(pintype "bidirectional+no_connect")
 		)
 		(pad "39" smd rect
@@
 			(layers "F.Cu" "F.Mask" "F.Paste")
 			(roundrect_rratio 0.25)
-			(net 30 "/MOTOR_IN1")
+			(net 31 "unconnected-(U2-PH{slash}IN2-Pad12)")
 			(pinfunction "PH/IN2")
-			(pintype "input")
+			(pintype "input+no_connect")
 		)
 		(pad "13" smd roundrect
@@
 			(layers "F.Cu" "F.Mask" "F.Paste")
 			(roundrect_rratio 0.25)
-			(net 31 "/MOTOR_IN2")
+			(net 30 "unconnected-(U2-EN{slash}IN1-Pad13)")
 			(pinfunction "EN/IN1")
-			(pintype "input")
+			(pintype "input+no_connect")
 		)
 		(pad "14" smd roundrect
@@
 	)
 	(segment
-		(start 102.77 116.07)
-		(end 103.95 114.89)
-		(width 0.2032)
-		(layer "F.Cu")
-		(net 30)
-	)
-	(segment
-		(start 101.5252 116.07)
-		(end 102.77 116.07)
-		(width 0.2032)
-		(layer "F.Cu")
-		(net 30)
-	)
-	(segment
-		(start 97.56673 116.17327)
-		(end 97.64 116.1)
-		(width 0.2032)
-		(layer "F.Cu")
-		(net 30)
-	)
-	(segment
-		(start 96.995 116.17327)
-		(end 97.56673 116.17327)
-		(width 0.2032)
-		(layer "F.Cu")
-		(net 30)
-	)
-	(via
-		(at 103.95 114.89)
-		(size 0.6)
-		(drill 0.3)
-		(layers "F.Cu" "B.Cu")
-		(net 30)
-	)
-	(via
-		(at 103.82 79.85)
-		(size 0.6)
-		(drill 0.3)
-		(layers "F.Cu" "B.Cu")
-		(net 30)
-	)
-	(via
-		(at 101.5252 116.07)
-		(size 0.6)
-		(drill 0.3)
-		(layers "F.Cu" "B.Cu")
-		(net 30)
-	)
-	(via
-		(at 97.64 116.1)
-		(size 0.6)
-		(drill 0.3)
-		(layers "F.Cu" "B.Cu")
-		(net 30)
-	)
-	(segment
-		(start 105.4734 81.5034)
-		(end 103.82 79.85)
-		(width 0.2032)
-		(layer "B.Cu")
-		(net 30)
-	)
-	(segment
-		(start 101.4952 116.1)
-		(end 101.5252 116.07)
-		(width 0.2032)
-		(layer "B.Cu")
-		(net 30)
-	)
-	(segment
-		(start 105.4734 113.3666)
-		(end 105.4734 81.5034)
-		(width 0.2032)
-		(layer "B.Cu")
-		(net 30)
-	)
-	(segment
-		(start 103.95 114.89)
-		(end 105.4734 113.3666)
-		(width 0.2032)
-		(layer "B.Cu")
-		(net 30)
-	)
-	(segment
-		(start 97.64 116.1)
-		(end 101.4952 116.1)
-		(width 0.2032)
-		(layer "B.Cu")
-		(net 30)
-	)
-	(segment
-		(start 92.928489 115.571222)
-		(end 92.729711 115.77)
-		(width 0.2032)
-		(layer "F.Cu")
-		(net 31)
-	)
-	(segment
-		(start 96.74577 115.46577)
-		(end 96.75 115.47)
-		(width 0.2032)
-		(layer "F.Cu")
-		(net 31)
-	)
-	(segment
-		(start 88.428051 81.921173)
-		(end 87.746878 81.24)
-		(width 0.2032)
-		(layer "F.Cu")
-		(net 31)
-	)
-	(segment
-		(start 87.746878 81.24)
-		(end 87.25 81.24)
-		(width 0.2032)
-		(layer "F.Cu")
-		(net 31)
-	)
-	(segment
-		(start 94.113519 115.571222)
-		(end 92.928489 115.571222)
-		(width 0.2032)
-		(layer "F.Cu")
-		(net 31)
-	)
-	(segment
-		(start 96.2875 115.46577)
-		(end 96.74577 115.46577)
-		(width 0.2032)
-		(layer "F.Cu")
-		(net 31)
-	)
-	(via
-		(at 92.729711 115.77)
-		(size 0.6)
-		(drill 0.3)
-		(layers "F.Cu" "B.Cu")
-		(net 31)
-	)
-	(via
-		(at 96.75 115.47)
-		(size 0.6)
-		(drill 0.3)
-		(layers "F.Cu" "B.Cu")
-		(net 31)
-	)
-	(via
-		(at 94.113519 115.571222)
-		(size 0.6)
-		(drill 0.3)
-		(layers "F.Cu" "B.Cu")
-		(net 31)
-	)
-	(via
-		(at 88.428051 81.921173)
-		(size 0.6)
-		(drill 0.3)
-		(layers "F.Cu" "B.Cu")
-		(net 31)
-	)
-	(segment
-		(start 90.08 98.94)
-		(end 90.08 83.573122)
-		(width 0.2032)
-		(layer "B.Cu")
-		(net 31)
-	)
-	(segment
-		(start 90.102849 98.962849)
-		(end 90.08 98.94)
-		(width 0.2032)
-		(layer "B.Cu")
-		(net 31)
-	)
-	(segment
-		(start 96.75 115.47)
-		(end 96.648778 115.571222)
-		(width 0.2032)
-		(layer "B.Cu")
-		(net 31)
-	)
-	(segment
-		(start 90.08 83.573122)
-		(end 88.428051 81.921173)
-		(width 0.2032)
-		(layer "B.Cu")
-		(net 31)
-	)
-	(segment
-		(start 92.68 115.77)
-		(end 90.102849 113.192849)
-		(width 0.2032)
-		(layer "B.Cu")
-		(net 31)
-	)
-	(segment
-		(start 90.102849 113.192849)
-		(end 90.102849 98.962849)
-		(width 0.2032)
-		(layer "B.Cu")
-		(net 31)
-	)
-	(segment
-		(start 92.729711 115.77)
-		(end 92.68 115.77)
-		(width 0.2032)
-		(layer "B.Cu")
-		(net 31)
-	)
-	(segment
-		(start 96.648778 115.571222)
-		(end 94.113519 115.571222)
-		(width 0.2032)
-		(layer "B.Cu")
-		(net 31)
-	)
-	(segment
