File: hardware/sounddecoder-esp32-s3-wroom-2-micro/sounddecoder-esp32-s3-wroom-2-micro.kicad_sch (KiCad schematic)
At the start: 48 parts, among them J1 Pins, J2 Conn_01x02_Pin, J3 TrackRight, J4 Smoke_Pin, J5 TrackLeft, U1 TPS54302, U2 DRV8235, U3 MAX98357A, U7 ESP32-S3-WROOM-2, U8 ULN2003A

Commit message: Added support of DRV8235 motor driver
Connections:
- net MOTOR_IN1: no longer names the net of U2.12 (PH/IN2)
- net MOTOR_IN1: no longer U7.38 (IO2)
- net MOTOR_IN2: no longer names the net of U2.13 (EN/IN1)
- net MOTOR_IN2: no longer U7.4 (IO4)
- no-connect marks 14 -> 18
Changed lines of the file:
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@@
+	)
+	(no_connect
+		(at 165.1 34.29)
 	)
 	(no_connect
@@
 	)
 	(no_connect
+		(at 168.91 109.22)
+	)
+	(no_connect
 		(at 168.91 124.46)
 	)
@@
 	)
 	(no_connect
+		(at 168.91 104.14)
+	)
+	(no_connect
 		(at 168.91 160.02)
+	)
+	(no_connect
+		(at 165.1 31.75)
 	)
 	(no_connect
@@
 	(wire
 		(pts
-			(xy 148.59 34.29) (xy 165.1 34.29)
-		)
-		(stroke
-			(width 0)
-			(type default)
-		)
-	)
-	(wire
-		(pts
 			(xy 165.1 60.96) (xy 165.1 58.42)
 		)
@@
 		(pts
 			(xy 156.21 127) (xy 168.91 127)
-		)
-		(stroke
-			(width 0)
-			(type default)
-		)
-	)
-	(wire
-		(pts
-			(xy 148.59 31.75) (xy 165.1 31.75)
 		)
 		(stroke
@@
 		)
 	)
-	(label "MOTOR_IN1"
-		(at 151.13 31.75 0)
-		(effects
-			(font
-				(size 1.27 1.27)
-			)
-			(justify left bottom)
-		)
-	)
 	(label "UART-TX{slash}GPIO A"
 		(at 157.48 167.64 0)
@@
 		)
 	)
-	(label "MOTOR_IN2"
-		(at 151.13 34.29 0)
-		(effects
-			(font
-				(size 1.27 1.27)
-			)
-			(justify left bottom)
-		)
-	)
 	(label "DCC"
 		(at 157.48 111.76 0)
@@
 		)
 	)
-	(label "MOTOR_IN2"
-		(at 157.48 109.22 0)
-		(effects
-			(font
-				(size 1.27 1.27)
-			)
-			(justify left bottom)
-		)
-	)
 	(label "SDA"
 		(at 199.39 40.64 0)
@@
 		(effects
 			(font
-				(size 1.27 1.27)
-			)
-			(justify left bottom)
-		)
-	)
-	(label "MOTOR_IN1"
-		(at 157.48 104.14 0)
-		(effects
-			(font
